File: PCB Design/9Key/Keypad.kicad_sch (KiCad schematic)
At the start: 30 parts, among them SW0 RotaryEncoder_Switch, SW1 SW_Push, SW2 SW_Push, SW3 SW_Push, SW4 SW_Push, SW5 SW_Push, SW6 SW_Push, SW7 SW_Push, SW8 SW_Push, SW9 SW_Push, U1 XIAO-RP2040-DIP

Commit message: Update
Connections:
- net 3V3: now also O1.2 (Pin_2); no longer O1.1 (Pin_1)
- net GND: now also O1.1 (Pin_1); no longer O1.2 (Pin_2)
Changed lines of the file:
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@@
 	(symbol
 		(lib_id "power:VCC")
-		(at 204.47 30.48 90)
+		(at 204.47 33.02 90)
 		(unit 1)
 		(exclude_from_sim no)
@@
 		(dnp no)
 		(property "Reference" "#PWR08"
-			(at 208.28 30.48 0)
+			(at 208.28 33.02 0)
 			(effects
 				(font
@@
 		)
 		(property "Value" "3V3"
-			(at 199.39 30.48 90)
+			(at 199.39 33.02 90)
 			(effects
 				(font
@@
 		)
 		(property "Footprint" ""
-			(at 204.47 30.48 0)
+			(at 204.47 33.02 0)
 			(effects
 				(font
@@
 		)
 		(property "Datasheet" ""
-			(at 204.47 30.48 0)
+			(at 204.47 33.02 0)
 			(effects
 				(font
@@
 		)
 		(property "Description" "Power symbol creates a global label with name \"VCC\""
-			(at 204.47 30.48 0)
+			(at 204.47 33.02 0)
 			(effects
 				(font
@@
 	(symbol
 		(lib_id "power:GND")
-		(at 204.47 33.02 270)
+		(at 204.47 30.48 270)
 		(unit 1)
 		(exclude_from_sim no)
@@
 		(dnp no)
 		(property "Reference" "#PWR07"
-			(at 198.12 33.02 0)
+			(at 198.12 30.48 0)
 			(effects
 				(font
@@
 		)
 		(property "Value" "GND"
-			(at 201.422 33.02 90)
+			(at 201.422 30.48 90)
 			(effects
 				(font
@@
 		)
 		(property "Footprint" ""
-			(at 204.47 33.02 0)
+			(at 204.47 30.48 0)
 			(effects
 				(font
@@
 		)
 		(property "Datasheet" ""
-			(at 204.47 33.02 0)
+			(at 204.47 30.48 0)
 			(effects
 				(font
@@
 		)
 		(property "Description" "Power symbol creates a global label with name \"GND\" , ground"
-			(at 204.47 33.02 0)
-			(effects
-				(font
+			(at 204.47 30.48 0)
+			(effects
+				(font
