File: PCB Design/9Key/Keypad.kicad_pcb (KiCad board)
At the start: 2 copper layers, 68 x 84 mm, 32 parts, among them SW0 RotaryEncoder_Switch, SW1 SW_Push, SW2 SW_Push, SW3 SW_Push, SW4 SW_Push, SW5 SW_Push, SW6 SW_Push, SW7 SW_Push, SW8 SW_Push, SW9 SW_Push, U1 XIAO-RP2040-DIP

Commit message: Update
Connections:
- O1 pad 1: 3V3 -> GND
- O1 pad 2: GND -> 3V3
Routing:
- net 3V3: track 23.7 -> 22.7 mm
- net GND: track 20.3 -> 19.3 mm
Other:
- board text added: "XIAO HERE!"
Changed lines of the file:
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@@
 	)
 	(setup
+		(stackup
+			(layer "F.SilkS"
+				(type "Top Silk Screen")
+			)
+			(layer "F.Paste"
+				(type "Top Solder Paste")
+			)
+			(layer "F.Mask"
+				(type "Top Solder Mask")
+				(thickness 0.01)
+			)
+			(layer "F.Cu"
+				(type "copper")
+				(thickness 0.035)
+			)
+			(layer "dielectric 1"
+				(type "core")
+				(thickness 1.51)
+				(material "FR4")
+				(epsilon_r 4.5)
+				(loss_tangent 0.02)
+			)
+			(layer "B.Cu"
+				(type "copper")
+				(thickness 0.035)
+			)
+			(layer "B.Mask"
+				(type "Bottom Solder Mask")
+				(thickness 0.01)
+			)
+			(layer "B.Paste"
+				(type "Bottom Solder Paste")
+			)
+			(layer "B.SilkS"
+				(type "Bottom Silk Screen")
+			)
+			(copper_finish "None")
+			(dielectric_constraints no)
+		)
 		(pad_to_mask_clearance 0)
 		(allow_soldermask_bridges_in_footprints no)
@@
 			(drillshape 0)
 			(scaleselection 1)
-			(outputdirectory "")
+			(outputdirectory "../../Production Files/Gerbers/")
 		)
 	)
@@
 			(net 19 "unconnected-(LED9-DOUT-Pad1)")
 			(pinfunction "DOUT")
-			(pintype "output")
+			(pintype "output+no_connect")
 		)
 		(pad "2" smd rect
@@
 			(pinfunction "VSS")
 			(pintype "power_in")
+			(thermal_bridge_width 0.25)
 		)
 		(pad "3" smd rect
@@
 			(pinfunction "VDD")
 			(pintype "power_in")
+			(thermal_bridge_width 0.25)
 		)
 		(embedded_fonts no)
@@
 		(tags "rotary encoder")
 		(property "Reference" "SW0"
-			(at 2.8 -4.7 0)
+			(at 11.5 -4.7 0)
 			(layer "F.SilkS")
 			(effects
@@
 			(net 24 "unconnected-(SW0-PadS1)")
 			(pinfunction "S1")
-			(pintype "passive")
+			(pintype "passive+no_connect")
 		)
 		(pad "S2" thru_hole circle
@@
 			(net 23 "unconnected-(SW0-PadS2)")
 			(pinfunction "S2")
-			(pintype "passive")
+			(pintype "passive+no_connect")
 		)
 		(embedded_fonts no)
@@
 			(at 1.9 5.91 90)
 			(layer "F.SilkS")
+			(hide yes)
 			(effects
 				(font
@@
 		)
 		(property "Value" "OLED"
-			(at 18.5 14 0)
+			(at 26.4 14.5 0)
 			(layer "F.Fab")
+			(hide yes)
 			(effects
 				(font
@@
 		)
 		(fp_text user "OLED Panel"
-			(at 19 6 0)
+			(at 39.4 6 90)
 			(layer "F.SilkS")
 			(effects
@@
 			(layers "*.Cu" "*.Mask")
 			(remove_unused_layers no)
-			(net 28 "3V3")
+			(net 1 "GND")
 			(pinfunction "Pin_1")
 			(pintype "passive")
@@
 			(layers "*.Cu" "*.Mask")
 			(remove_unused_layers no)
-			(net 1 "GND")
+			(net 28 "3V3")
 			(pinfunction "Pin_2")
 			(pintype "passive")
@@
 		(layer "Edge.Cuts")
 	)
+	(gr_text "XIAO HERE!"
+		(at 151 62 0)
+		(layer "B.SilkS")
+		(effects
+			(font
+				(size 1 1)
+				(thickness 0.1)
+			)
+			(justify left bottom mirror)
+		)
+	)
 	(segment
 		(start 130.875 129.125)
 		(end 131 129)
-		(width 0.2)
+		(width 0.5)
 		(layer "F.Cu")
 		(net 1)
@@
 	(segment
 		(start 167 91)
-		(end 168 91)
-		(width 0.2)
+		(end 169 91)
+		(width 0.5)
 		(layer "F.Cu")
 		(net 1)
@@
 		(start 129 110.125)
 		(end 130.875 110.125)
-		(width 0.2)
+		(width 0.5)
 		(layer "F.Cu")
 		(net 1)
@@
 		(start 144.25 92.875)
 		(end 144.25 93.75)
-		(width 0.2)
+		(width 0.5)
 		(layer "F.Cu")
 		(net 1)
@@
 		(start 168.75 129.25)
 		(end 169 129)
-		(width 0.2)
+		(width 0.5)
 		(layer "F.Cu")
 		(net 1)
@@
 		(start 144.25 130.875)
 		(end 142.875 130.875)
-		(width 0.2)
-		(layer "F.Cu")
-		(net 1)
-	)
-	(segment
-		(start 167 91)
-		(end 169 91)
-		(width 0.2)
+		(width 0.5)
 		(layer "F.Cu")
 		(net 1)
@@
 		(start 166.75 110.125)
 		(end 168.875 110.125)
-		(width 0.2)
+		(width 0.5)
 		(layer "F.Cu")
 		(net 1)
@@
 		(start 128.75 129.125)
 		(end 130.875 129.125)
-		(width 0.2)
+		(width 0.5)
 		(layer "F.Cu")
 		(net 1)
@@
 		(start 144.25 93.75)
 		(end 144 94)
-		(width 0.2)
+		(width 0.5)
 		(layer "F.Cu")
 		(net 1)
@@
 		(start 144.25 113.75)
 		(end 144 114)
-		(width 0.2)
+		(width 0.5)
 		(layer "F.Cu")
 		(net 1)
@@
 		(start 168.875 110.125)
 		(end 169 110)
-		(width 0.2)
+		(width 0.5)
 		(layer "F.Cu")
 		(net 1)
@@
 		(start 128.75 91.125)
 		(end 131.875 91.125)
-		(width 0.2)
+		(width 0.5)
 		(layer "F.Cu")
 		(net 1)
@@
 		(start 144.25 112.75)
 		(end 144.25 113.75)
-		(width 0.2)
+		(width 0.5)
 		(layer "F.Cu")
 		(net 1)
@@
 		(start 142.875 130.875)
 		(end 142 130)
-		(width 0.2)
+		(width 0.5)
 		(layer "F.Cu")
 		(net 1)
@@
 		(start 167 129.25)
 		(end 168.75 129.25)
-		(width 0.2)
+		(width 0.5)
 		(layer "F.Cu")
 		(net 1)
@@
 		(start 131.875 91.125)
 		(end 132 91)
-		(width 0.2)
+		(width 0.5)
 		(layer "F.Cu")
 		(net 1)
@@
 		(start 130.875 110.125)
 		(end 131 110)
-		(width 0.2)
+		(width 0.5)
 		(layer "F.Cu")
 		(net 1)
@@
 	(via
 		(at 131 129)
-		(size 0.6)
-		(drill 0.3)
+		(size 1)
+		(drill 0.5)
 		(layers "F.Cu" "B.Cu")
 		(net 1)
@@
 	(via
 		(at 131 110)
-		(size 0.6)
-		(drill 0.3)
+		(size 1)
+		(drill 0.5)
 		(layers "F.Cu" "B.Cu")
 		(net 1)
@@
 	(via
 		(at 169 110)
-		(size 0.6)
-		(drill 0.3)
+		(size 1)
+		(drill 0.5)
 		(layers "F.Cu" "B.Cu")
 		(net 1)
@@
 	(via
 		(at 144 94)
-		(size 0.6)
-		(drill 0.3)
+		(size 1)
+		(drill 0.5)
 		(layers "F.Cu" "B.Cu")
 		(net 1)
@@
 	(via
 		(at 169 91)
-		(size 0.6)
-		(drill 0.3)
+		(size 1)
+		(drill 0.5)
 		(layers "F.Cu" "B.Cu")
 		(net 1)
@@
 	(via
 		(at 144 114)
-		(size 0.6)
-		(drill 0.3)
+		(size 1)
+		(drill 0.5)
 		(layers "F.Cu" "B.Cu")
 		(net 1)
@@
 	(via
 		(at 132 91)
-		(size 0.6)
-		(drill 0.3)
+		(size 1)
+		(drill 0.5)
 		(layers "F.Cu" "B.Cu")
 		(net 1)
@@
 	(via
 		(at 142 130)
-		(size 0.6)
-		(drill 0.3)
+		(size 1)
+		(drill 0.5)
 		(layers "F.Cu" "B.Cu")
 		(net 1)
@@
 	(via
 		(at 169 129)
-		(size 0.6)
-		(drill 0.3)
+		(size 1)
+		(drill 0.5)
 		(layers "F.Cu" "B.Cu")
 		(net 1)
@@
 	)
 	(segment
-		(start 138.38 58.08)
-		(end 129.13 58.08)
-		(width 0.2)
+		(start 118.9 65.77)
+		(end 126.59 58.08)
+		(width 0.5)
 		(layer "F.Cu")
 		(net 28)
 	)
 	(segment
-		(start 129.13 58.08)
-		(end 118.9 68.31)
-		(width 0.2)
+		(start 126.59 58.08)
+		(end 138.38 58.08)
+		(width 0.5)
 		(layer "F.Cu")
 		(net 28)

Commit message: uPDATE
Parts:
- removed the REF** at (176.0, 54.0)
- removed the REF** at (116.0, 54.0)
- added REF**: MountingHole_3.2mm_M3, MountingHole:MountingHole_3.2mm_M3, F.Cu at (116.0, 130.0)
- added REF**: MountingHole_3.2mm_M3, MountingHole:MountingHole_3.2mm_M3, F.Cu at (176.0, 130.0)
- moved SW0 4.03 mm to (158.0, 58.0)
- moved O1 2.50 mm to (155.4, 68.0)
Routing:
- net Net-(U1-GPIO28/ADC2/A2): track 14.6 -> 8.66 mm
- net Net-(U1-GPIO29/ADC3/A3): track 4.45 -> 5.76 mm
- net Net-(O1-Pin_4): track 44.1 -> 43.1 mm
- net Net-(O1-Pin_3): track 45.9 -> 44.9 mm
- net 3V3: track 22.7 -> 21.6 mm
- net Net-(D3-K): track 120.9 -> 121.9 mm
- net Net-(D2-K): track 101.0 -> 102.0 mm

Commit message: Assembly
Parts:
- moved O1 5.08 mm to (154.5, 63.0)
- moved SW0 5.02 mm to (157.5, 53.0)
- moved U1 2.12 mm to (146.0, 58.5)
Routing:
- net Net-(D2-K): track 102.0 -> 108.4 mm
- net Net-(D3-K): track 121.9 -> 126.6 mm
- net Net-(U1-GPIO28/ADC2/A2): track 8.66 -> 4.72 mm
- net Net-(U1-GPIO2/SCK): track 54.2 -> 56.4 mm
- net Net-(U1-GPIO3/MOSI): track 64.1 -> 66.2 mm
- net Net-(LED1-DIN): track 28.3 -> 30.4 mm
- net Net-(D1-K): track 67.9 -> 70.1 mm
- net Net-(U1-GPIO29/ADC3/A3): track 5.76 -> 7.40 mm
- net Net-(U1-GPIO4/MISO): track 68.0 -> 68.9 mm
Other:
- board size 68 x 84 mm -> 68 x 86 mm
